File: cerberus/hardware-4.0/doorctrl-v4-gpio.sch (KiCad schematic (older format))
At the start: 33 parts, among them CON3 RJHSE-5085, CON4 RJHSE-5085, CON5 RJHSE-5085, K1 G5SB, K2 CONN_3_V, K3 CONN_3_V, K4 G5SB, P1 CONN_2_V, Q3 BC817, Q4 BC817

Commit message: Misc labeling
git-svn-id: file:///home/ff/projects/osaa/svn@219 a092026d-3e22-4cff-94a7-eaa6fdd35d37
Other:
- note added: "R22 and R23 must NOT be mounted along with the on-board RFID reader."
Changed lines of the file:
@@
-EESchema Schematic File Version 2  date 2010-12-17T21:22:49 CET
+EESchema Schematic File Version 2  date 2010-12-17T21:31:15 CET
 LIBS:enc28j60
 LIBS:power
@@
 EELAYER END
 $Descr A4 11700 8267
-Sheet 3 6
+Sheet 4 6
 Title ""
 Date "17 dec 2010"
@@
 Comment4 ""
 $EndDescr
+Text Notes 1550 6950 0    60   ~ 0
+R22 and R23 must NOT be mounted along with the on-board RFID reader.
 Wire Wire Line
 	8950 4400 8950 4650
@@
 Relay2
 $Comp
-L GND #PWR71
+L GND #PWR69
 U 1 1 4D07A06D
 P 8950 5950
-F 0 "#PWR71" H 8950 5950 30  0001 C CNN
+F 0 "#PWR69" H 8950 5950 30  0001 C CNN
 F 1 "GND" H 8950 5880 30  0001 C CNN
 	1    8950 5950
@@
 $EndComp
 $Comp
-L +12V #PWR70
+L +12V #PWR68
 U 1 1 4D07A02C
 P 8950 4400
-F 0 "#PWR70" H 8950 4350 20  0001 C CNN
+F 0 "#PWR68" H 8950 4350 20  0001 C CNN
 F 1 "+12V" H 8950 4500 30  0000 C CNN
 	1    8950 4400
@@
 $EndComp
 $Comp
-L +12V #PWR68
+L +12V #PWR66
 U 1 1 4D079D91
 P 8950 2300
-F 0 "#PWR68" H 8950 2250 20  0001 C CNN
+F 0 "#PWR66" H 8950 2250 20  0001 C CNN
 F 1 "+12V" H 8950 2400 30  0000 C CNN
 	1    8950 2300
@@
 $EndComp
 $Comp
-L GND #PWR69
+L GND #PWR67
 U 1 1 4D079B9C
 P 8950 3900
-F 0 "#PWR69" H 8950 3900 30  0001 C CNN
+F 0 "#PWR67" H 8950 3900 30  0001 C CNN
 F 1 "GND" H 8950 3830 30  0001 C CNN
 	1    8950 3900
@@
 $EndComp
 $Comp
-L GND #PWR67
+L GND #PWR65
 U 1 1 4D04DDDA
 P 8150 1950
-F 0 "#PWR67" H 8150 1950 30  0001 C CNN
+F 0 "#PWR65" H 8150 1950 30  0001 C CNN
 F 1 "GND" H 8150 1880 30  0001 C CNN
 	1    8150 1950
@@
 $EndComp
 $Comp
-L +12V #PWR66
+L +12V #PWR64
 U 1 1 4D04DDD3
 P 8150 1450
-F 0 "#PWR66" H 8150 1400 20  0001 C CNN
+F 0 "#PWR64" H 8150 1400 20  0001 C CNN
 F 1 "+12V" H 8150 1550 30  0000 C CNN
 	1    8150 1450
@@
 port3-1d
 $Comp
-L GND #PWR65
+L GND #PWR63
 U 1 1 4D04BA37
 P 2850 6550
-F 0 "#PWR65" H 2850 6550 30  0001 C CNN
+F 0 "#PWR63" H 2850 6550 30  0001 C CNN
 F 1 "GND" H 2850 6480 30  0001 C CNN
 	1    2850 6550
@@
 port3-1
 $Comp
-L +12V #PWR62
+L +12V #PWR60
 U 1 1 4D04B962
 P 2750 6150
-F 0 "#PWR62" H 2750 6100 20  0001 C CNN
+F 0 "#PWR60" H 2750 6100 20  0001 C CNN
 F 1 "+12V" H 2750 6250 30  0000 C CNN
 	1    2750 6150
@@
 $EndComp
 $Comp
-L +12V #PWR60
+L +12V #PWR58
 U 1 1 4D04A9E3
 P 2700 4100
-F 0 "#PWR60" H 2700 4050 20  0001 C CNN
+F 0 "#PWR58" H 2700 4050 20  0001 C CNN
 F 1 "+12V" H 2700 4200 30  0000 C CNN
 	1    2700 4100
@@
 $EndComp
 $Comp
-L GND #PWR64
+L GND #PWR62
 U 1 1 4D04A9DA
 P 2850 4500
-F 0 "#PWR64" H 2850 4500 30  0001 C CNN
+F 0 "#PWR62" H 2850 4500 30  0001 C CNN
 F 1 "GND" H 2850 4430 30  0001 C CNN
 	1    2850 4500
@@
 $EndComp
 $Comp
-L +12V #PWR61
+L +12V #PWR59
 U 1 1 4D04A4F5
 P 2750 2400
-F 0 "#PWR61" H 2750 2350 20  0001 C CNN
+F 0 "#PWR59" H 2750 2350 20  0001 C CNN
 F 1 "+12V" H 2750 2500 30  0000 C CNN
 	1    2750 2400
@@
 $EndComp
 $Comp
-L GND #PWR63
+L GND #PWR61
 U 1 1 4D04A4D9
 P 2850 2800
-F 0 "#PWR63" H 2850 2800 30  0001 C CNN
+F 0 "#PWR61" H 2850 2800 30  0001 C CNN
 F 1 "GND" H 2850 2730 30  0001 C CNN
 	1    2850 2800
