File: cerberus/hardware-4.0/doorctrl-v4-gpio.sch (KiCad schematic (older format))
At the start: 33 parts, among them CON3 RJHSE-5085, CON4 RJHSE-5085, CON5 RJHSE-5085, K1 G5SB, K2 CONN_3_V, K3 CONN_3_V, K4 G5SB, P1 CONN_2_V, Q3 BC817, Q4 BC817

Commit message: Added torroid coil and proper diode packages
git-svn-id: file:///home/ff/projects/osaa/svn@222 a092026d-3e22-4cff-94a7-eaa6fdd35d37
Connections:
- net labels added: k1a, k1b, k1c, k4a, k4b, k4c
Changed lines of the file:
@@
-EESchema Schematic File Version 2  date 2010-12-18T14:49:05 CET
+EESchema Schematic File Version 2  date 2010-12-19T21:45:09 CET
 LIBS:enc28j60
 LIBS:power
@@
 Sheet 4 6
 Title ""
-Date "18 dec 2010"
+Date "19 dec 2010"
 Rev ""
 Comp ""
@@
 Comment4 ""
 $EndDescr
+Text Label 8050 2800 0    60   ~ 0
+k1c
+Text Label 8250 3000 0    60   ~ 0
+k1b
+Text Label 8250 2600 0    60   ~ 0
+k1a
+Text Label 8050 4850 0    60   ~ 0
+k4c
+Text Label 8250 5050 0    60   ~ 0
+k4b
+Text Label 8250 4650 0    60   ~ 0
+k4a
 Text Notes 1550 6950 0    60   ~ 0
 R22 and R23 must NOT be mounted along with the on-board RFID reader.
@@
 	5450 3800 5450 4200
 Wire Wire Line
-	6250 4150 6250 4600
+	6250 4600 6250 4150
 Wire Wire Line
 	5450 3400 5450 3500
@@
 	1800 2000 2000 2000
 Wire Wire Line
-	6250 4600 5200 4600
+	5200 4600 6250 4600
 Wire Wire Line
 	8050 2700 8250 2700
@@
 Relay2
 $Comp
-L GND #PWR69
+L GND #PWR046
 U 1 1 4D07A06D
 P 8950 5950
-F 0 "#PWR69" H 8950 5950 30  0001 C CNN
+F 0 "#PWR046" H 8950 5950 30  0001 C CNN
 F 1 "GND" H 8950 5880 30  0001 C CNN
 	1    8950 5950
@@
 $EndComp
 $Comp
-L +12V #PWR68
+L +12V #PWR047
 U 1 1 4D07A02C
 P 8950 4400
-F 0 "#PWR68" H 8950 4350 20  0001 C CNN
+F 0 "#PWR047" H 8950 4350 20  0001 C CNN
 F 1 "+12V" H 8950 4500 30  0000 C CNN
 	1    8950 4400
@@
 F 1 "CONN_3_V" H 7700 5040 40  0000 C CNN
 	1    7700 4850
-	-1   0    0    1
+	-1   0    0    -1
 $EndComp
 $Comp
@@
 F 1 "CONN_3_V" H 7700 2990 40  0000 C CNN
 	1    7700 2800
-	-1   0    0    1
-$EndComp
-$Comp
-L +12V #PWR66
+	-1   0    0    -1
+$EndComp
+$Comp
+L +12V #PWR048
 U 1 1 4D079D91
 P 8950 2300
-F 0 "#PWR66" H 8950 2250 20  0001 C CNN
+F 0 "#PWR048" H 8950 2250 20  0001 C CNN
 F 1 "+12V" H 8950 2400 30  0000 C CNN
 	1    8950 2300
@@
 $EndComp
 $Comp
-L GND #PWR67
+L GND #PWR049
 U 1 1 4D079B9C
 P 8950 3900
-F 0 "#PWR67" H 8950 3900 30  0001 C CNN
+F 0 "#PWR049" H 8950 3900 30  0001 C CNN
 F 1 "GND" H 8950 3830 30  0001 C CNN
 	1    8950 3900
@@
 $EndComp
 $Comp
-L GND #PWR65
+L GND #PWR050
 U 1 1 4D04DDDA
 P 8150 1950
-F 0 "#PWR65" H 8150 1950 30  0001 C CNN
+F 0 "#PWR050" H 8150 1950 30  0001 C CNN
 F 1 "GND" H 8150 1880 30  0001 C CNN
 	1    8150 1950
@@
 $EndComp
 $Comp
-L +12V #PWR64
+L +12V #PWR051
 U 1 1 4D04DDD3
 P 8150 1450
-F 0 "#PWR64" H 8150 1400 20  0001 C CNN
+F 0 "#PWR051" H 8150 1400 20  0001 C CNN
 F 1 "+12V" H 8150 1550 30  0000 C CNN
 	1    8150 1450
@@
 port3-1d
 $Comp
-L GND #PWR63
+L GND #PWR052
 U 1 1 4D04BA37
 P 2850 6550
-F 0 "#PWR63" H 2850 6550 30  0001 C CNN
+F 0 "#PWR052" H 2850 6550 30  0001 C CNN
 F 1 "GND" H 2850 6480 30  0001 C CNN
 	1    2850 6550
@@
 port3-1
 $Comp
-L +12V #PWR60
+L +12V #PWR053
 U 1 1 4D04B962
 P 2750 6150
-F 0 "#PWR60" H 2750 6100 20  0001 C CNN
+F 0 "#PWR053" H 2750 6100 20  0001 C CNN
 F 1 "+12V" H 2750 6250 30  0000 C CNN
 	1    2750 6150
@@
 $EndComp
 $Comp
-L +12V #PWR58
+L +12V #PWR054
 U 1 1 4D04A9E3
 P 2700 4100
-F 0 "#PWR58" H 2700 4050 20  0001 C CNN
+F 0 "#PWR054" H 2700 4050 20  0001 C CNN
 F 1 "+12V" H 2700 4200 30  0000 C CNN
 	1    2700 4100
@@
 $EndComp
 $Comp
-L GND #PWR62
+L GND #PWR055
 U 1 1 4D04A9DA
 P 2850 4500
-F 0 "#PWR62" H 2850 4500 30  0001 C CNN
+F 0 "#PWR055" H 2850 4500 30  0001 C CNN
 F 1 "GND" H 2850 4430 30  0001 C CNN
 	1    2850 4500
@@
 $EndComp
 $Comp
-L +12V #PWR59
+L +12V #PWR056
 U 1 1 4D04A4F5
 P 2750 2400
-F 0 "#PWR59" H 2750 2350 20  0001 C CNN
+F 0 "#PWR056" H 2750 2350 20  0001 C CNN
 F 1 "+12V" H 2750 2500 30  0000 C CNN
 	1    2750 2400
@@
 $EndComp
 $Comp
-L GND #PWR61
+L GND #PWR057
 U 1 1 4D04A4D9
 P 2850 2800
-F 0 "#PWR61" H 2850 2800 30  0001 C CNN
+F 0 "#PWR057" H 2850 2800 30  0001 C CNN
 F 1 "GND" H 2850 2730 30  0001 C CNN
 	1    2850 2800

Commit message: Started laying out the PCB for real
git-svn-id: file:///home/ff/projects/osaa/svn@223 a092026d-3e22-4cff-94a7-eaa6fdd35d37
Parts:
- removed D6, D7: DIODE, symbol DIODE
- removed Q3, Q4: BC817, symbol NPN
- added D10, D11: LS 914B, diode-MINIMELF, symbol DIODE-MINIMELF
- added Q3, Q4: BC817, symbol BC817
Connections:
- net labels added: k2a, k2b, k2c
- net labels removed: k1a, k1b, k1c
- wire segments 99 -> 103
Changed lines of the file:
@@
-EESchema Schematic File Version 2  date 2010-12-19T21:45:09 CET
+EESchema Schematic File Version 2  date 2010-12-20T22:26:04 CET
 LIBS:enc28j60
 LIBS:power
@@
 LIBS:linear
 LIBS:atmel
+LIBS:diode
 LIBS:doorctrl-v4-cache
 EELAYER 24  0
@@
 Sheet 4 6
 Title ""
-Date "19 dec 2010"
+Date "20 dec 2010"
 Rev ""
 Comp ""
@@
 Comment4 ""
 $EndDescr
-Text Label 8050 2800 0    60   ~ 0
-k1c
-Text Label 8250 3000 0    60   ~ 0
-k1b
-Text Label 8250 2600 0    60   ~ 0
-k1a
-Text Label 8050 4850 0    60   ~ 0
+Text Label 8100 4850 0    60   ~ 0
 k4c
 Text Label 8250 5050 0    60   ~ 0
@@
 Text Label 8250 4650 0    60   ~ 0
 k4a
-Text Notes 1550 6950 0    60   ~ 0
-R22 and R23 must NOT be mounted along with the on-board RFID reader.
+Text Label 8100 2800 0    60   ~ 0
+k2c
+Text Label 8250 3000 0    60   ~ 0
+k2b
+Text Label 8250 2600 0    60   ~ 0
+k2a
+$Comp
+L BC817 Q4
+U 1 1 4D0FB782
+P 9050 5450
+F 0 "Q4" H 9050 5300 50  0000 R CNN
+F 1 "BC817" H 9050 5600 50  0000 R CNN
+	1    9050 5450
+	-1   0    0    -1
+$EndComp
+$Comp
+L BC817 Q3
+U 1 1 4D0FB771
+P 9050 3400
+F 0 "Q3" H 9050 3250 50  0000 R CNN
+F 1 "BC817" H 9050 3550 50  0000 R CNN
+	1    9050 3400
+	-1   0    0    -1
+$EndComp
+Wire Wire Line
+	9300 4950 9300 5050
+Wire Wire Line
+	9300 2900 9300 3000
 Wire Wire Line
 	8950 4400 8950 4650
@@
 	8950 3200 8950 3000
 Wire Wire Line
-	9300 2600 8950 2600
+	8950 2600 9300 2600
 Wire Wire Line
 	8550 3000 8250 3000
@@
 	5450 3800 5450 4200
 Wire Wire Line
-	6250 4600 6250 4150
+	6250 4150 6250 4600
 Wire Wire Line
 	5450 3400 5450 3500
@@
 	1800 2000 2000 2000
 Wire Wire Line
-	5200 4600 6250 4600
+	6250 4600 5200 4600
 Wire Wire Line
 	8050 2700 8250 2700
@@
 Wire Wire Line
 	8950 4650 9300 4650
+Wire Wire Line
+	9300 2600 9300 2700
+Wire Wire Line
+	9300 4650 9300 4750
+$Comp
+L DIODE-MINIMELF D11
+U 1 1 4D0FB50F
+P 9300 4850
+F 0 "D11" H 9400 4869 50  0000 L BNN
+F 1 "LS 914B" H 9400 4759 50  0000 L BNN
+F 2 "diode-MINIMELF" H 9300 5000 50  0001 C CNN
+	1    9300 4850
+	0    -1   -1   0
+$EndComp
+$Comp
+L DIODE-MINIMELF D10
+U 1 1 4D0FB4EA
+P 9300 2800
+F 0 "D10" H 9400 2819 50  0000 L BNN
+F 1 "LS 914B" H 9400 2709 50  0000 L BNN
+F 2 "diode-MINIMELF" H 9300 2950 50  0001 C CNN
+	1    9300 2800
+	0    -1   -1   0
+$EndComp
+Text Notes 1550 6950 0    60   ~ 0
+R22 and R23 must NOT be mounted along with the on-board RFID reader.
 Text HLabel 10150 5450 2    60   Input ~ 0
 Relay2
@@
 	1    9750 5450
 	0    1    1    0
-$EndComp
-$Comp
-L NPN Q4
-U 1 1 4D07A03F
-P 9050 5450
-F 0 "Q4" H 9050 5300 50  0000 R CNN
-F 1 "BC817" H 9050 5600 50  0000 R CNN
-	1    9050 5450
-	-1   0    0    -1
-$EndComp
-$Comp
-L DIODE D7
-U 1 1 4D07A035
-P 9300 4850
-F 0 "D7" H 9300 4950 40  0000 C CNN
-F 1 "DIODE" H 9300 4750 40  0000 C CNN
-	1    9300 4850
-	0    -1   -1   0
 $EndComp
 $Comp
@@
 $EndComp
 $Comp
-L NPN Q3
-U 1 1 4D079B69
-P 9050 3400
-F 0 "Q3" H 9050 3250 50  0000 R CNN
-F 1 "BC817" H 9050 3550 50  0000 R CNN
-	1    9050 3400
-	-1   0    0    -1
-$EndComp
-$Comp
-L DIODE D6
-U 1 1 4D079B5D
-P 9300 2800
-F 0 "D6" H 9300 2900 40  0000 C CNN
-F 1 "DIODE" H 9300 2700 40  0000 C CNN
-	1    9300 2800
-	0    -1   -1   0
-$EndComp
-$Comp

Commit message: Did some silk work
git-svn-id: file:///home/ff/projects/osaa/svn@231 a092026d-3e22-4cff-94a7-eaa6fdd35d37
Connections:
- net GND: now also CON3.22 (shield), CON4.22 (shield), CON5.22 (shield)
Changed lines of the file:
@@
-EESchema Schematic File Version 2  date 2010-12-23T21:46:15 CET
+EESchema Schematic File Version 2  date 2010-12-25T12:56:58 CET
 LIBS:enc28j60
 LIBS:power
@@
 Sheet 4 6
 Title ""
-Date "23 dec 2010"
+Date "25 dec 2010"
 Rev ""
 Comp ""
@@
 Comment4 ""
 $EndDescr
+Connection ~ 2850 6600
+Wire Wire Line
+	2850 6350 2850 6700
+Connection ~ 2850 4550
+Wire Wire Line
+	2850 4650 2850 4300
+Connection ~ 2850 2850
+Wire Wire Line
+	2850 2950 2850 2600
 Wire Wire Line
 	9300 4950 9300 5050
@@
 Connection ~ 2850 6450
 Wire Wire Line
-	2850 6350 2850 6550
-Wire Wire Line
 	2000 6250 1800 6250
 Wire Wire Line
@@
 Connection ~ 2850 2700
 Wire Wire Line
-	2850 2800 2850 2600
-Wire Wire Line
 	2850 2400 2850 2300
 Wire Wire Line
@@
 Wire Wire Line
 	2500 4200 2850 4200
-Wire Wire Line
-	2850 4300 2850 4500
 Connection ~ 2850 4400
 Wire Wire Line
@@
 L GND #PWR052
 U 1 1 4D04BA37
-P 2850 6550
-F 0 "#PWR052" H 2850 6550 30  0001 C CNN
-F 1 "GND" H 2850 6480 30  0001 C CNN
-	1    2850 6550
+P 2850 6700
+F 0 "#PWR052" H 2850 6700 30  0001 C CNN
+F 1 "GND" H 2850 6630 30  0001 C CNN
+	1    2850 6700
 	1    0    0    -1
 $EndComp
@@
 L GND #PWR055
 U 1 1 4D04A9DA
-P 2850 4500
-F 0 "#PWR055" H 2850 4500 30  0001 C CNN
-F 1 "GND" H 2850 4430 30  0001 C CNN
-	1    2850 4500
+P 2850 4650
+F 0 "#PWR055" H 2850 4650 30  0001 C CNN
+F 1 "GND" H 2850 4580 30  0001 C CNN
+	1    2850 4650
 	1    0    0    -1
 $EndComp
@@
 L GND #PWR057
 U 1 1 4D04A4D9
-P 2850 2800
-F 0 "#PWR057" H 2850 2800 30  0001 C CNN
-F 1 "GND" H 2850 2730 30  0001 C CNN
-	1    2850 2800
-	1    0    0    -1
-$EndComp
+P 2850 2950
+F 0 "#PWR057" H 2850 2950 30  0001 C CNN
+F 1 "GND" H 2850 2880 30  0001 C CNN
+	1    2850 2950
+	1    0    0    -1
+$EndComp
