File: cerberus/hardware-4.0/doorctrl-v4-psu.sch (KiCad schematic (older format))
At the start: 0 parts

Commit message: Did more kicad migration, still not yet complete schematic
git-svn-id: file:///home/ff/projects/osaa/svn@207 a092026d-3e22-4cff-94a7-eaa6fdd35d37
Parts:
- added C10: 1200uF, symbol CAPAPOL
- added C11: 2.2nF, symbol C
- added C12: 33nF, symbol C
- added C13: 2.2uF, symbol C
- added C14: 1000uF, symbol CAPAPOL
- added C15, C17: 100uF, symbol CAPAPOL
- added C16, C19, C20, C21, C22, C23, C24, C25, C26, C27, C28, C29: 100nF, symbol C
- added C18: 10uF, symbol C
- added C9: 82pF, symbol C
- added D2: SK 86, symbol DIODESCH
- added D3: SK 34SMA, symbol DIODESCH
- added L1: 220uH, symbol INDUCTOR
- added L2: 330uH, symbol INDUCTOR
- added R26, R30: 4k7, symbol R
- added R27: 0.22R, symbol R
- added R28: 15k, symbol R
- added R29: 6k2, symbol R
- added R31: 11k, symbol R
- added R32: 18k, symbol R
- added U2: MC34063, symbol MC34063
- added U3: L4960, l4960-HEPTAWATT, symbol L4960
Connections:
- net labels added: +12V, +24V, +3.3V, GND
- wire segments 0 -> 42
Other:
- note added: "Distributed decoupling capacitors"
