File: cerberus/hardware-4.0/doorctrl-v4.sch (KiCad schematic (older format))
At the start: 6 parts, among them CON1 AVR-ISP-6, CON2 AVR-JTAG-10, IC1 ATMEGA324P-A, X1 12 MHz

Commit message: Did more kicad migration, still not yet complete schematic
git-svn-id: file:///home/ff/projects/osaa/svn@207 a092026d-3e22-4cff-94a7-eaa6fdd35d37
Connections:
- wire segments 66 -> 69
Changed lines of the file:
@@
-EESchema Schematic File Version 2  date 2010-12-07T16:59:15 CET
+EESchema Schematic File Version 2  date 2010-12-12T18:56:18 CET
 LIBS:power
 LIBS:device
@@
 LIBS:bc807
 LIBS:bc817
+LIBS:amp-rj45-tap-up-with-leds
+LIBS:l4960
+LIBS:borniers
+LIBS:doorctrl-v4-cache
 EELAYER 24  0
 EELAYER END
@@
 Sheet 1 6
 Title ""
-Date "7 dec 2010"
+Date "12 dec 2010"
 Rev ""
 Comp ""
@@
 Comment4 ""
 $EndDescr
+Wire Wire Line
+	4250 3350 6100 3350
+Wire Wire Line
+	1850 2350 1850 2475
+Wire Wire Line
+	1150 1950 1050 1950
+Wire Wire Line
+	4150 4450 4225 4450
+Wire Wire Line
+	4150 4250 4225 4250
+Wire Wire Line
+	4150 4050 4225 4050
+Wire Wire Line
+	4150 3850 4225 3850
+Wire Wire Line
+	4150 3550 4225 3550
+Wire Wire Line
+	4150 3350 4225 3350
+Wire Wire Line
+	4150 3050 4225 3050
+Wire Wire Line
+	4150 2450 4225 2450
+Wire Wire Line
+	4150 2350 4225 2350
+Wire Wire Line
+	4150 2150 4225 2150
+Wire Wire Line
+	4150 2750 4225 2750
+Wire Wire Line
+	4150 2550 4225 2550
+Wire Wire Line
+	4150 1850 4225 1850
+Wire Wire Line
+	4150 1650 4225 1650
+Wire Wire Line
+	4150 1450 4225 1450
+Wire Wire Line
+	4150 1250 4225 1250
+Wire Wire Line
+	2150 2350 2150 2275
+Connection ~ 4225 3150
+Wire Wire Line
+	4150 3150 4225 3150
+Connection ~ 2750 5600
+Connection ~ 2750 5700
+Connection ~ 2750 5800
+Connection ~ 2750 6000
+Connection ~ 3675 6000
+Connection ~ 3825 5800
+Connection ~ 3675 5600
+Wire Wire Line
+	3675 5700 3300 5700
+Wire Wire Line
+	3050 5600 2750 5600
+Wire Wire Line
+	3050 5800 2750 5800
+Wire Wire Line
+	3050 6000 2750 6000
+Connection ~ 950  5600
+Connection ~ 950  5700
+Connection ~ 950  5800
+Connection ~ 1800 5800
+Connection ~ 1800 5700
+Wire Wire Line
+	1250 5800 950  5800
+Wire Wire Line
+	1250 5600 950  5600
+Connection ~ 3000 775
+Wire Wire Line
+	3000 775  3000 850
+Wire Wire Line
+	3300 850  3300 775
+Wire Wire Line
+	3300 775  2800 775
+Wire Wire Line
+	2800 775  2800 850
+Connection ~ 3000 4950
+Wire Wire Line
+	3000 4950 3000 4850
+Wire Wire Line
+	3200 4850 3200 4950
+Wire Wire Line
+	3200 4950 2900 4950
+Wire Wire Line
+	2900 4950 2900 4850
+Wire Wire Line
+	1500 5700 1800 5700
+Wire Wire Line
+	1500 5600 1800 5600
+Wire Wire Line
+	1500 5800 1800 5800
+Wire Wire Line
+	3100 4950 3100 4850
+Connection ~ 3100 4950
+Wire Wire Line
+	3050 4950 3050 5075
+Connection ~ 3050 4950
+Wire Wire Line
+	2900 850  2900 775
+Connection ~ 2900 775
+Wire Wire Line
+	3125 775  3125 675
+Connection ~ 3125 775
+Wire Wire Line
+	1250 5700 950  5700
+Wire Wire Line
+	3300 5800 3825 5800
+Wire Wire Line
+	3300 6000 3675 6000
+Wire Wire Line
+	3050 5700 2750 5700
+Wire Wire Line
+	3675 5600 3300 5600
+Wire Wire Line
+	2150 1150 2100 1150
+Wire Wire Line
+	4150 1150 4225 1150
+Wire Wire Line
+	4150 1350 4225 1350
+Wire Wire Line
+	4150 1550 4225 1550
+Wire Wire Line
+	4150 1750 4225 1750
+Wire Wire Line
+	4150 2650 4225 2650
+Wire Wire Line
+	4150 2050 4225 2050
+Wire Wire Line
+	4150 2250 4225 2250
+Wire Wire Line
+	4150 2950 4225 2950
+Wire Wire Line
+	4150 3250 4225 3250
+Wire Wire Line
+	4150 3450 4225 3450
+Wire Wire Line
+	4150 3650 4225 3650
+Wire Wire Line
+	4150 3950 4225 3950
+Wire Wire Line
+	4150 4150 4225 4150
+Wire Wire Line
+	4150 4350 4225 4350
+Wire Wire Line
+	4150 4550 4225 4550
+Connection ~ 4225 1150
+Connection ~ 4225 1250
+Connection ~ 4225 1350
+Connection ~ 4225 1450
+Connection ~ 4225 1550
+Connection ~ 4225 1650
+Connection ~ 4225 1750
+Connection ~ 4225 1850
+Connection ~ 4225 2050
+Connection ~ 4225 2150
+Connection ~ 4225 2250
+Connection ~ 4225 2350
+Connection ~ 4225 2450
+Connection ~ 4225 2550
+Connection ~ 4225 2650
+Connection ~ 4225 2750
+Connection ~ 4225 2950
+Connection ~ 4225 3050
+Connection ~ 4225 3250
+Connection ~ 4225 3350
+Connection ~ 4225 3450
+Connection ~ 4225 3550
+Connection ~ 4225 3650
+Connection ~ 4225 3850
+Connection ~ 4225 3950
+Connection ~ 4225 4050
+Connection ~ 4225 4150
+Connection ~ 4225 4250
+Connection ~ 4225 4350
+Connection ~ 4225 4450
+Connection ~ 4225 4550
+Connection ~ 2100 1150
+Connection ~ 2100 1950
+Wire Wire Line
+	1750 1950 2150 1950
+Connection ~ 1850 1950
+Wire Wire Line
+	1050 1950 1050 1550
+Wire Wire Line
+	1050 1550 2150 1550
+Wire Wire Line
+	1050 2350 1050 2475
+Connection ~ 1050 1950
+Wire Wire Line
+	4250 3450 6100 3450
+Wire Wire Line
+	4250 3250 6100 3250
 $Sheet
 S 6100 800  1200 5000
@@
 F0 "doorctrl-v4-gpio" 60
 F1 "doorctrl-v4-gpio.sch" 60
+F2 "port3-2d" I R 7300 5650 60
+F3 "port3-1d" I R 7300 5500 60
+F4 "LED-3" I L 6100 3250 60
+F5 "LED-2" I L 6100 3350 60
+F6 "LED-1" I L 6100 3450 60
 $EndSheet
 $Sheet
@@
 $EndSheet
 $Sheet
-S 9300 800  1600 1050
+S 9300 800  1600 1000
 U 4CFD3054
 F0 "doorctrl-v4-psu" 60
@@
 	1    0    0    -1
 $EndComp
-Connection ~ 1050 1950
-Wire Wire Line
-	1050 2350 1050 2475
-Wire Wire Line
-	2150 1550 1050 1550
-Wire Wire Line
-	1050 1550 1050 1950
-Connection ~ 1850 1950
-Wire Wire Line
-	1750 1950 2150 1950
-Connection ~ 2100 1950
-Connection ~ 2100 1150
-Connection ~ 4225 4550
-Connection ~ 4225 4450
-Connection ~ 4225 4350
-Connection ~ 4225 4250
-Connection ~ 4225 4150
-Connection ~ 4225 4050
-Connection ~ 4225 3950
-Connection ~ 4225 3850
-Connection ~ 4225 3650
-Connection ~ 4225 3550
-Connection ~ 4225 3450
-Connection ~ 4225 3350
-Connection ~ 4225 3250
-Connection ~ 4225 3050
-Connection ~ 4225 2950
-Connection ~ 4225 2750
-Connection ~ 4225 2650
-Connection ~ 4225 2550
-Connection ~ 4225 2450
-Connection ~ 4225 2350
-Connection ~ 4225 2250
-Connection ~ 4225 2150
-Connection ~ 4225 2050
-Connection ~ 4225 1850
-Connection ~ 4225 1750
-Connection ~ 4225 1650
-Connection ~ 4225 1550
-Connection ~ 4225 1450
-Connection ~ 4225 1350
-Connection ~ 4225 1250
-Connection ~ 4225 1150
-Wire Wire Line
-	4150 4550 4225 4550
-Wire Wire Line
-	4150 4350 4225 4350
-Wire Wire Line
-	4150 4150 4225 4150
-Wire Wire Line
-	4150 3950 4225 3950
-Wire Wire Line
-	4150 3650 4225 3650
-Wire Wire Line
-	4150 3450 4225 3450
-Wire Wire Line
-	4150 3250 4225 3250
-Wire Wire Line
-	4150 2950 4225 2950
-Wire Wire Line
-	4150 2250 4225 2250
-Wire Wire Line
-	4150 2050 4225 2050
-Wire Wire Line
-	4150 2650 4225 2650
-Wire Wire Line
-	4150 1750 4225 1750
-Wire Wire Line
-	4150 1550 4225 1550
-Wire Wire Line
-	4150 1350 4225 1350
-Wire Wire Line
-	4150 1150 4225 1150
-Wire Wire Line
-	2150 1150 2100 1150
-Wire Wire Line
-	3675 5600 3300 5600
-Wire Wire Line
-	3050 5700 2750 5700
-Wire Wire Line
-	3300 6000 3675 6000
-Wire Wire Line
-	3300 5800 3825 5800
-Wire Wire Line
-	1250 5700 950  5700
-Connection ~ 3125 775
-Wire Wire Line
-	3125 775  3125 675
-Connection ~ 2900 775
-Wire Wire Line
-	2900 850  2900 775
-Connection ~ 3050 4950
-Wire Wire Line
-	3050 4950 3050 5075
-Connection ~ 3100 4950
-Wire Wire Line
-	3100 4950 3100 4850
-Wire Wire Line
-	1500 5800 1800 5800
-Wire Wire Line
-	1500 5600 1800 5600
-Wire Wire Line
-	1500 5700 1800 5700
-Wire Wire Line
-	2900 4850 2900 4950
-Wire Wire Line
-	2900 4950 3200 4950
-Wire Wire Line
-	3200 4950 3200 4850
-Wire Wire Line
-	3000 4950 3000 4850
-Connection ~ 3000 4950
-Wire Wire Line
-	2800 850  2800 775
-Wire Wire Line
-	2800 775  3300 775
-Wire Wire Line
-	3300 775  3300 850
-Wire Wire Line
-	3000 775  3000 850
-Connection ~ 3000 775
-Wire Wire Line
-	1250 5600 950  5600
-Wire Wire Line
-	1250 5800 950  5800
-Connection ~ 1800 5700
-Connection ~ 1800 5800
-Connection ~ 950  5800
-Connection ~ 950  5700
-Connection ~ 950  5600
-Wire Wire Line
-	3050 6000 2750 6000
-Wire Wire Line
-	3050 5800 2750 5800
-Wire Wire Line
-	3050 5600 2750 5600
-Wire Wire Line
-	3675 5700 3300 5700
-Connection ~ 3675 5600
-Connection ~ 3825 5800
-Connection ~ 3675 6000
-Connection ~ 2750 6000
-Connection ~ 2750 5800
-Connection ~ 2750 5700
-Connection ~ 2750 5600
-Wire Wire Line
-	4150 3150 4225 3150
-Connection ~ 4225 3150
-Wire Wire Line
-	2150 2350 2150 2275
-Wire Wire Line
-	4150 1250 4225 1250
-Wire Wire Line
-	4150 1450 4225 1450
-Wire Wire Line
-	4150 1650 4225 1650
-Wire Wire Line
-	4150 1850 4225 1850
-Wire Wire Line
-	4150 2550 4225 2550
-Wire Wire Line
-	4150 2750 4225 2750
-Wire Wire Line
-	4150 2150 4225 2150
-Wire Wire Line
-	4150 2350 4225 2350
-Wire Wire Line
-	4150 2450 4225 2450
-Wire Wire Line
-	4150 3050 4225 3050
-Wire Wire Line
-	4150 3350 4225 3350
-Wire Wire Line
-	4150 3550 4225 3550
-Wire Wire Line
-	4150 3850 4225 3850
-Wire Wire Line
-	4150 4050 4225 4050
-Wire Wire Line
-	4150 4250 4225 4250
-Wire Wire Line
-	4150 4450 4225 4450
-Wire Wire Line
-	1050 1950 1150 1950
-Wire Wire Line
-	1850 2350 1850 2475
 $Comp
 L GND #PWR02

Commit message: Blaarghle
git-svn-id: file:///home/ff/projects/osaa/svn@212 a092026d-3e22-4cff-94a7-eaa6fdd35d37
Changed lines of the file:
@@
-EESchema Schematic File Version 2  date 2010-12-13T21:30:20 CET
+EESchema Schematic File Version 2  date 2010-12-14T20:47:45 CET
+LIBS:enc28j60
 LIBS:power
 LIBS:device
@@
 EELAYER END
 $Descr A4 11700 8267
-Sheet 1 6
+Sheet 1 5
 Title ""
-Date "13 dec 2010"
+Date "14 dec 2010"
 Rev ""
 Comp ""
@@
 	4250 3250 6100 3250
 $Sheet
-S 6100 800  1200 5000
+S 6100 800  950  3850
 U 4CFD3197
 F0 "doorctrl-v4-gpio" 60
 F1 "doorctrl-v4-gpio.sch" 60
-F2 "port3-2d" I R 7300 5650 60
-F3 "port3-1d" I R 7300 5500 60
+F2 "port3-2d" I R 7050 3650 60
+F3 "port3-1d" I R 7050 3550 60
 F4 "LED-3" I L 6100 3250 60
 F5 "LED-2" I L 6100 3350 60
 F6 "LED-1" I L 6100 3450 60
+F7 "Relay2" I L 6100 3000 60
+F8 "Relay1" I L 6100 2900 60
+F9 "port3-6" I L 6100 2800 60
+F10 "port3-3" I L 6100 2700 60
+F11 "port3-2" I L 6100 2600 60
+F12 "port3-1" I L 6100 2500 60
+F13 "port2-6" I L 6100 2300 60
+F14 "port2-3" I L 6100 2200 60
+F15 "port2-2" I L 6100 2100 60
+F16 "port2-1" I L 6100 2000 60
+F17 "port1-6" I L 6100 1800 60
+F18 "port1-3" I L 6100 1700 60
+F19 "port1-2" I L 6100 1600 60
+F20 "port1-1" I L 6100 1500 60
 $EndSheet
 $Sheet
-S 9300 2100 1600 1100
-U 4CFD3096
-F0 "doorctrl-v4-relays" 60
-F1 "doorctrl-v4-relays.sch" 60
-$EndSheet
-$Sheet
-S 9300 4850 1600 1000
+S 9300 3400 1600 1000
 U 4CFD3072
 F0 "doorctrl-v4-rfid" 60
 F1 "doorctrl-v4-rfid.sch" 60
-F2 "RFID" O L 9300 5300 60
-F3 "Coil-B" B L 9300 5500 60
-F4 "Coil-A" B L 9300 5650 60
-F5 "Carrier" I L 9300 5100 60
+F2 "RFID" O L 9300 3850 60
+F3 "Coil-B" B L 9300 4050 60
+F4 "Coil-A" B L 9300 4200 60
+F5 "Carrier" I L 9300 3650 60
 $EndSheet
 $Sheet
@@
 $EndSheet
 $Sheet
-S 9300 3450 1600 1100
+S 9300 2100 1600 1100
 U 4CFD2FB8
-F0 "doorctrl-v4-ethernet" 60
-F1 "doorctrl-v4-ethernet.sch" 60
+F0 "doorctrl-v4-net" 60
+F1 "doorctrl-v4-net.sch" 60
 $EndSheet
 NoConn ~ 3300 5900
@@
 PB5
 $Comp
-L +3.3V #PWR4
+L +3.3V #PWR01
 U 1 1 4CFAB301
 P 2150 2275
-F 0 "#PWR4" H 2150 2235 30  0001 C CNN
+F 0 "#PWR01" H 2150 2235 30  0001 C CNN
 F 1 "+3.3V" H 2150 2385 30  0000 C CNN
 	1    2150 2275
@@
 $EndComp
 $Comp
-L GND #PWR3
+L GND #PWR02
 U 1 1 4CFAB0A0
 P 1850 2475
-F 0 "#PWR3" H 1850 2475 30  0001 C CNN
+F 0 "#PWR02" H 1850 2475 30  0001 C CNN
 F 1 "GND" H 1850 2405 30  0001 C CNN
 	1    1850 2475
@@
 $EndComp
 $Comp
-L GND #PWR1
+L GND #PWR03
 U 1 1 4CFAB098
 P 1050 2475
-F 0 "#PWR1" H 1050 2475 30  0001 C CNN
+F 0 "#PWR03" H 1050 2475 30  0001 C CNN
 F 1 "GND" H 1050 2405 30  0001 C CNN
 	1    1050 2475
@@
 PC2
 $Comp
-L +3.3V #PWR7
+L +3.3V #PWR04
 U 1 1 4CFA7FD7
 P 3675 5700
-F 0 "#PWR7" H 3675 5660 30  0001 C CNN
+F 0 "#PWR04" H 3675 5660 30  0001 C CNN
 F 1 "+3.3V" H 3675 5810 30  0000 C CNN
 	1    3675 5700
@@
 $EndComp
 $Comp
-L +3.3V #PWR2
+L +3.3V #PWR05
 U 1 1 4CFA5CC7
 P 1800 5600
-F 0 "#PWR2" H 1800 5560 30  0001 C CNN
+F 0 "#PWR05" H 1800 5560 30  0001 C CNN
 F 1 "+3.3V" H 1800 5710 30  0000 C CNN
 	1    1800 5600
@@
 RESET
 $Comp
-L GND #PWR5
+L GND #PWR06
 U 1 1 4CF6BFD7
 P 3050 5075
-F 0 "#PWR5" H 3050 5075 30  0001 C CNN
+F 0 "#PWR06" H 3050 5075 30  0001 C CNN
 F 1 "GND" H 3050 5005 30  0001 C CNN
 	1    3050 5075
@@
 $EndComp
 $Comp
-L +3.3V #PWR6
+L +3.3V #PWR07
 U 1 1 4CF6BFC6
 P 3125 675
-F 0 "#PWR6" H 3125 635 30  0001 C CNN
+F 0 "#PWR07" H 3125 635 30  0001 C CNN
 F 1 "+3.3V" H 3125 785 30  0000 C CNN
 	1    3125 675
