File: cerberus/hardware-4.0/doorctrl-v4-rfid.sch (KiCad schematic (older format))
At the start: 19 parts, among them Q1 BC817, Q2 BC807, U1 LM358

Commit message: Added a 5V regulator for most stuff, except ENC28J60 which lives on its own 3.3v supply
git-svn-id: file:///home/ff/projects/osaa/svn@217 a092026d-3e22-4cff-94a7-eaa6fdd35d37
Connections:
- net +3.3V renamed +5V
Changed lines of the file:
@@
-EESchema Schematic File Version 2  date 2010-12-16T22:33:40 CET
+EESchema Schematic File Version 2  date 2010-12-17T21:22:49 CET
 LIBS:enc28j60
 LIBS:power
@@
 LIBS:pulse-pe-68517-ethernet-trafo
 LIBS:sn65hvd1x
+LIBS:i2c
 LIBS:doorctrl-v4-cache
 EELAYER 24  0
 EELAYER END
 $Descr A4 11700 8267
-Sheet 3 5
+Sheet 4 6
 Title ""
-Date "16 dec 2010"
+Date "17 dec 2010"
 Rev ""
 Comp ""
@@
 Comment4 ""
 $EndDescr
+$Comp
+L +5V #PWR58
+U 1 1 4D0BAFCB
+P 9150 2650
+F 0 "#PWR58" H 9150 2740 20  0001 C CNN
+F 1 "+5V" H 9150 2740 30  0000 C CNN
+	1    9150 2650
+	1    0    0    -1
+$EndComp
+$Comp
+L +5V #PWR55
+U 1 1 4D0BAFC8
+P 7250 2550
+F 0 "#PWR55" H 7250 2640 20  0001 C CNN
+F 1 "+5V" H 7250 2640 30  0000 C CNN
+	1    7250 2550
+	1    0    0    -1
+$EndComp
+$Comp
+L +5V #PWR47
+U 1 1 4D0BAFBC
+P 2950 2550
+F 0 "#PWR47" H 2950 2640 20  0001 C CNN
+F 1 "+5V" H 2950 2640 30  0000 C CNN
+	1    2950 2550
+	1    0    0    -1
+$EndComp
 $Comp
 L BC807 Q2
@@
 Carrier
 $Comp
-L GND #PWR51
+L GND #PWR57
 U 1 1 4CFD37F8
 P 8650 3850
-F 0 "#PWR51" H 8650 3850 30  0001 C CNN
+F 0 "#PWR57" H 8650 3850 30  0001 C CNN
 F 1 "GND" H 8650 3780 30  0001 C CNN
 	1    8650 3850
@@
 $EndComp
 $Comp
-L GND #PWR48
+L GND #PWR54
 U 1 1 4CFD37F3
 P 6850 4600
-F 0 "#PWR48" H 6850 4600 30  0001 C CNN
+F 0 "#PWR54" H 6850 4600 30  0001 C CNN
 F 1 "GND" H 6850 4530 30  0001 C CNN
 	1    6850 4600
@@
 $EndComp
 $Comp
-L GND #PWR47
+L GND #PWR53
 U 1 1 4CFD37EF
 P 6450 4200
-F 0 "#PWR47" H 6450 4200 30  0001 C CNN
+F 0 "#PWR53" H 6450 4200 30  0001 C CNN
 F 1 "GND" H 6450 4130 30  0001 C CNN
 	1    6450 4200
@@
 $EndComp
 $Comp
-L GND #PWR46
+L GND #PWR52
 U 1 1 4CFD37EC
 P 6150 4200
-F 0 "#PWR46" H 6150 4200 30  0001 C CNN
+F 0 "#PWR52" H 6150 4200 30  0001 C CNN
 F 1 "GND" H 6150 4130 30  0001 C CNN
 	1    6150 4200
@@
 $EndComp
 $Comp
-L GND #PWR45
+L GND #PWR51
 U 1 1 4CFD37E8
 P 4800 4200
-F 0 "#PWR45" H 4800 4200 30  0001 C CNN
+F 0 "#PWR51" H 4800 4200 30  0001 C CNN
 F 1 "GND" H 4800 4130 30  0001 C CNN
 	1    4800 4200
@@
 $EndComp
 $Comp
-L GND #PWR44
+L GND #PWR50
 U 1 1 4CFD37E5
 P 4300 4200
-F 0 "#PWR44" H 4300 4200 30  0001 C CNN
+F 0 "#PWR50" H 4300 4200 30  0001 C CNN
 F 1 "GND" H 4300 4130 30  0001 C CNN
 	1    4300 4200
@@
 $EndComp
 $Comp
-L GND #PWR43
+L GND #PWR49
 U 1 1 4CFD37E2
 P 3600 4200
-F 0 "#PWR43" H 3600 4200 30  0001 C CNN
+F 0 "#PWR49" H 3600 4200 30  0001 C CNN
 F 1 "GND" H 3600 4130 30  0001 C CNN
 	1    3600 4200
@@
 $EndComp
 $Comp
-L +3.3V #PWR49
-U 1 1 4CFD37DA
-P 7250 2550
-F 0 "#PWR49" H 7250 2510 30  0001 C CNN
-F 1 "+3.3V" H 7250 2660 30  0000 C CNN
-	1    7250 2550
-	1    0    0    -1
-$EndComp
-$Comp
-L +3.3V #PWR52
-U 1 1 4CFD37D2
-P 9150 2650
-F 0 "#PWR52" H 9150 2610 30  0001 C CNN
-F 1 "+3.3V" H 9150 2760 30  0000 C CNN
-	1    9150 2650
-	1    0    0    -1
-$EndComp
-$Comp
-L GND #PWR53
+L GND #PWR59
 U 1 1 4CFD37CF
 P 9150 3550
-F 0 "#PWR53" H 9150 3550 30  0001 C CNN
+F 0 "#PWR59" H 9150 3550 30  0001 C CNN
 F 1 "GND" H 9150 3480 30  0001 C CNN
 	1    9150 3550
@@
 $EndComp
 $Comp
-L GND #PWR50
+L GND #PWR56
 U 1 1 4CFD37C7
 P 7250 3450
-F 0 "#PWR50" H 7250 3450 30  0001 C CNN
+F 0 "#PWR56" H 7250 3450 30  0001 C CNN
 F 1 "GND" H 7250 3380 30  0001 C CNN
 	1    7250 3450
@@
 $EndComp
 $Comp
-L GND #PWR42
+L GND #PWR48
 U 1 1 4CFD378E
 P 2950 4200
-F 0 "#PWR42" H 2950 4200 30  0001 C CNN
+F 0 "#PWR48" H 2950 4200 30  0001 C CNN
 F 1 "GND" H 2950 4130 30  0001 C CNN
 	1    2950 4200
 	1    0    0    -1
 $EndComp
-$Comp
-L +3.3V #PWR41
-U 1 1 4CFD3789
-P 2950 2550
-F 0 "#PWR41" H 2950 2510 30  0001 C CNN
-F 1 "+3.3V" H 2950 2660 30  0000 C CNN
-	1    2950 2550
-	1    0    0    -1
-$EndComp
