File: cerberus/hardware-4.0/doorctrl-v4-rfid.sch (KiCad schematic (older format))
At the start: 19 parts, among them Q1 BC817, Q2 BC807, U1 LM358

Commit message: Started laying out the PCB for real
git-svn-id: file:///home/ff/projects/osaa/svn@223 a092026d-3e22-4cff-94a7-eaa6fdd35d37
Parts:
- removed D1: DIODE, symbol DIODE
- added D9: LS 914B, diode-MINIMELF, symbol DIODE-MINIMELF
Changed lines of the file:
@@
-EESchema Schematic File Version 2  date 2010-12-19T21:45:09 CET
+EESchema Schematic File Version 2  date 2010-12-20T22:26:04 CET
 LIBS:enc28j60
 LIBS:power
@@
 LIBS:linear
 LIBS:atmel
+LIBS:diode
 LIBS:doorctrl-v4-cache
 EELAYER 24  0
@@
 Sheet 5 6
 Title ""
-Date "19 dec 2010"
+Date "20 dec 2010"
 Rev ""
 Comp ""
@@
 Comment4 ""
 $EndDescr
+Wire Wire Line
+	4050 2900 5000 2900
+Wire Wire Line
+	4300 3750 4300 4200
+Wire Wire Line
+	9150 2650 9150 2700
+Wire Wire Line
+	7250 3450 7250 3400
+Wire Wire Line
+	8650 3750 8650 3850
+Wire Wire Line
+	8750 3200 8550 3200
+Wire Wire Line
+	9800 3100 9800 2400
+Wire Wire Line
+	9800 2400 9350 2400
+Wire Wire Line
+	8750 3000 8550 3000
+Wire Wire Line
+	7850 3000 8050 3000
+Wire Wire Line
+	7850 3000 7850 3950
+Wire Wire Line
+	7850 3950 7550 3950
+Connection ~ 6850 3950
+Wire Wire Line
+	6850 3100 6850 4000
+Wire Wire Line
+	6850 3700 7100 3700
+Wire Wire Line
+	6150 3700 6150 4200
+Connection ~ 6450 2900
+Wire Wire Line
+	6450 2900 6450 3250
+Wire Wire Line
+	5400 2900 5500 2900
+Connection ~ 4800 2900
+Wire Wire Line
+	4800 2900 4800 3300
+Wire Wire Line
+	3600 3600 3600 3700
+Connection ~ 3600 2900
+Wire Wire Line
+	3600 3100 3600 2900
+Connection ~ 2650 3200
+Wire Wire Line
+	2250 3200 2650 3200
+Wire Wire Line
+	2950 2550 2950 2700
+Wire Wire Line
+	2650 2900 2650 3500
+Wire Wire Line
+	2950 3300 2950 3100
+Wire Wire Line
+	2950 3700 2950 4200
+Wire Wire Line
+	3050 3200 2950 3200
+Connection ~ 2950 3200
+Wire Wire Line
+	3600 4100 3600 4200
+Connection ~ 4300 2900
+Wire Wire Line
+	4800 4200 4800 3800
+Wire Wire Line
+	6000 2900 6850 2900
+Wire Wire Line
+	6150 3300 6150 2900
+Connection ~ 6150 2900
+Wire Wire Line
+	6450 3750 6450 4200
+Wire Wire Line
+	6850 3950 7050 3950
+Connection ~ 6850 3700
+Wire Wire Line
+	6850 4500 6850 4600
+Wire Wire Line
+	7500 3700 7850 3700
+Connection ~ 7850 3700
+Wire Wire Line
+	8050 3000 8050 3200
+Connection ~ 7850 3000
+Connection ~ 8050 3000
+Wire Wire Line
+	8650 3000 8650 2400
+Wire Wire Line
+	8650 2400 8850 2400
+Connection ~ 8650 3000
+Wire Wire Line
+	9150 3500 9150 3550
+Wire Wire Line
+	8650 3200 8650 3350
+Connection ~ 8650 3200
+Wire Wire Line
+	9950 3100 9750 3100
+Connection ~ 9800 3100
+Wire Wire Line
+	7250 2550 7250 2600
+Wire Wire Line
+	4300 2900 4300 3350
+Wire Wire Line
+	3850 2900 3450 2900
+$Comp
+L DIODE-MINIMELF D9
+U 1 1 4D0FB594
+P 3950 2900
+F 0 "D9" H 4050 2919 50  0000 L BNN
+F 1 "LS 914B" H 3850 2750 50  0000 L BNN
+F 2 "diode-MINIMELF" H 3950 3050 50  0001 C CNN
+	1    3950 2900
+	1    0    0    -1
+$EndComp
 $Comp
 L +5V #PWR058
@@
 	1    0    0    -1
 $EndComp
-Wire Wire Line
-	4300 3750 4300 4200
-Wire Wire Line
-	9150 2650 9150 2700
-Wire Wire Line
-	7250 3450 7250 3400
-Wire Wire Line
-	8650 3750 8650 3850
-Wire Wire Line
-	8750 3200 8550 3200
-Wire Wire Line
-	9800 3100 9800 2400
-Wire Wire Line
-	9800 2400 9350 2400
-Wire Wire Line
-	8750 3000 8550 3000
-Wire Wire Line
-	7850 3000 8050 3000
-Wire Wire Line
-	7850 3000 7850 3950
-Wire Wire Line
-	7850 3950 7550 3950
-Connection ~ 6850 3950
-Wire Wire Line
-	6850 3100 6850 4000
-Wire Wire Line
-	6850 3700 7100 3700
-Wire Wire Line
-	6150 3700 6150 4200
-Connection ~ 6450 2900
-Wire Wire Line
-	6450 2900 6450 3250
-Wire Wire Line
-	5400 2900 5500 2900
-Connection ~ 4800 2900
-Wire Wire Line
-	4800 2900 4800 3300
-Wire Wire Line
-	3600 3600 3600 3700
-Connection ~ 3600 2900
-Wire Wire Line
-	3600 3100 3600 2900
-Connection ~ 2650 3200
-Wire Wire Line
-	2250 3200 2650 3200
-Wire Wire Line
-	2950 2550 2950 2700
-Wire Wire Line
-	2650 2900 2650 3500
-Wire Wire Line
-	2950 3300 2950 3100
-Wire Wire Line
-	2950 3700 2950 4200
-Wire Wire Line
-	3750 2900 3450 2900
-Wire Wire Line
-	3050 3200 2950 3200
-Connection ~ 2950 3200
-Wire Wire Line
-	3600 4100 3600 4200
-Wire Wire Line
-	4150 2900 5000 2900
-Connection ~ 4300 2900
-Wire Wire Line
-	4800 4200 4800 3800
-Wire Wire Line
-	6000 2900 6850 2900
-Wire Wire Line
-	6150 3300 6150 2900
-Connection ~ 6150 2900
-Wire Wire Line
-	6450 3750 6450 4200
-Wire Wire Line
-	6850 3950 7050 3950
-Connection ~ 6850 3700
-Wire Wire Line
-	6850 4500 6850 4600
-Wire Wire Line
-	7500 3700 7850 3700
-Connection ~ 7850 3700
-Wire Wire Line
-	8050 3000 8050 3200
-Connection ~ 7850 3000
-Connection ~ 8050 3000
-Wire Wire Line
-	8650 3000 8650 2400
-Wire Wire Line
-	8650 2400 8850 2400
-Connection ~ 8650 3000
-Wire Wire Line
-	9150 3500 9150 3550
-Wire Wire Line
-	8650 3200 8650 3350
-Connection ~ 8650 3200
-Wire Wire Line
-	9950 3100 9750 3100
-Connection ~ 9800 3100
-Wire Wire Line
-	7250 2550 7250 2600
-Wire Wire Line
-	4300 2900 4300 3350
 Text HLabel 9950 3100 2    60   Output ~ 0
 RFID
@@
 	1    0    0    -1
 $EndComp
-$Comp
-L DIODE D1
-U 1 1 4CFD360C
-P 3950 2900
-F 0 "D1" H 3950 3000 40  0000 C CNN
-F 1 "DIODE" H 3950 2800 40  0000 C CNN
-	1    3950 2900
-	1    0    0    -1
-$EndComp

Commit message: Finished the copper layers
git-svn-id: file:///home/ff/projects/osaa/svn@229 a092026d-3e22-4cff-94a7-eaa6fdd35d37
Connections:
- net Coil-A: now also D9.A, R1.1; no longer Q1.2 (E), Q2.2 (E)
- net Coil-B: now also Q1.2 (E), Q2.2 (E); no longer D9.A, R1.1
Changed lines of the file:
@@
-EESchema Schematic File Version 2  date 2010-12-21T17:47:20 CET
+EESchema Schematic File Version 2  date 2010-12-23T21:46:15 CET
 LIBS:enc28j60
 LIBS:power
@@
 LIBS:diode
 LIBS:doorctrl-v4-cache
-EELAYER 24  0
+EELAYER 25  0
 EELAYER END
 $Descr A4 11700 8267
 Sheet 5 6
 Title ""
-Date "21 dec 2010"
+Date "23 dec 2010"
 Rev ""
 Comp ""
@@
 Text HLabel 9950 3100 2    60   Output ~ 0
 RFID
+Text HLabel 3050 3200 2    60   BiDi ~ 0
+Coil-B
 Text HLabel 3450 2900 0    60   BiDi ~ 0
-Coil-B
-Text HLabel 3050 3200 2    60   BiDi ~ 0
 Coil-A
 Text HLabel 2250 3200 0    60   Input ~ 0
