File: cerberus/hardware-4.0/doorctrl-rs485.sch (KiCad schematic (older format))
At the start: 11 parts, among them CON7 RJHSE-5085, CON8 RJHSE-5085, U7 sp485

Commit message: Added torroid coil and proper diode packages
git-svn-id: file:///home/ff/projects/osaa/svn@222 a092026d-3e22-4cff-94a7-eaa6fdd35d37
Changed lines of the file:
@@
-EESchema Schematic File Version 2  date 2010-12-18T14:49:05 CET
+EESchema Schematic File Version 2  date 2010-12-19T21:45:09 CET
 LIBS:enc28j60
 LIBS:power
@@
 Sheet 3 6
 Title ""
-Date "18 dec 2010"
+Date "19 dec 2010"
 Rev ""
 Comp ""
@@
 $EndDescr
 $Comp
-L +5V #PWR74
+L +5V #PWR037
 U 1 1 4D0BB20A
 P 5450 2300
-F 0 "#PWR74" H 5450 2390 20  0001 C CNN
+F 0 "#PWR037" H 5450 2390 20  0001 C CNN
 F 1 "+5V" H 5450 2390 30  0000 C CNN
 	1    5450 2300
@@
 $EndComp
 $Comp
-L GND #PWR75
+L GND #PWR038
 U 1 1 4D0BB201
 P 5450 3400
-F 0 "#PWR75" H 5450 3400 30  0001 C CNN
+F 0 "#PWR038" H 5450 3400 30  0001 C CNN
 F 1 "GND" H 5450 3330 30  0001 C CNN
 	1    5450 3400
@@
 TXENABLE
 $Comp
-L +24V #PWR76
+L +24V #PWR039
 U 1 1 4D0BB200
 P 6150 4450
-F 0 "#PWR76" H 6150 4400 20  0001 C CNN
+F 0 "#PWR039" H 6150 4400 20  0001 C CNN
 F 1 "+24V" H 6150 4550 30  0000 C CNN
 	1    6150 4450
@@
 $EndComp
 $Comp
-L GND #PWR77
+L GND #PWR040
 U 1 1 4D0BB1FF
 P 6150 4900
-F 0 "#PWR77" H 6150 4900 30  0001 C CNN
+F 0 "#PWR040" H 6150 4900 30  0001 C CNN
 F 1 "GND" H 6150 4830 30  0001 C CNN
 	1    6150 4900
@@
 $EndComp
 $Comp
-L GND #PWR78
+L GND #PWR041
 U 1 1 4D0BB1FA
 P 7650 3250
-F 0 "#PWR78" H 7650 3250 30  0001 C CNN
+F 0 "#PWR041" H 7650 3250 30  0001 C CNN
 F 1 "GND" H 7650 3180 30  0001 C CNN
 	1    7650 3250
@@
 Termination jumpers
 $Comp
-L GND #PWR71
+L GND #PWR042
 U 1 1 4D0BB1F9
 P 4200 4150
-F 0 "#PWR71" H 4200 4150 30  0001 C CNN
+F 0 "#PWR042" H 4200 4150 30  0001 C CNN
 F 1 "GND" H 4200 4080 30  0001 C CNN
 	1    4200 4150
@@
 $EndComp
 $Comp
-L GND #PWR72
+L GND #PWR043
 U 1 1 4D0BB1F7
 P 4450 4150
-F 0 "#PWR72" H 4450 4150 30  0001 C CNN
+F 0 "#PWR043" H 4450 4150 30  0001 C CNN
 F 1 "GND" H 4450 4080 30  0001 C CNN
 	1    4450 4150
@@
 $EndComp
 $Comp
-L GND #PWR73
+L GND #PWR044
 U 1 1 4D0BB1F6
 P 4700 4150
-F 0 "#PWR73" H 4700 4150 30  0001 C CNN
+F 0 "#PWR044" H 4700 4150 30  0001 C CNN
 F 1 "GND" H 4700 4080 30  0001 C CNN
 	1    4700 4150
@@
 $EndComp
 $Comp
-L GND #PWR70
+L GND #PWR045
 U 1 1 4D0BB1F2
 P 3950 4150
-F 0 "#PWR70" H 3950 4150 30  0001 C CNN
+F 0 "#PWR045" H 3950 4150 30  0001 C CNN
 F 1 "GND" H 3950 4080 30  0001 C CNN
 	1    3950 4150
@@
 	7050 3000 6900 3000
 Wire Wire Line
-	7650 2700 7550 2700
-Wire Wire Line
-	7650 3250 7650 2700
+	7550 2700 7650 2700
+Wire Wire Line
+	7650 2700 7650 3250
 Connection ~ 6150 4500
 Wire Wire Line
 	6150 4450 6150 4500
 Wire Wire Line
-	4850 3100 4950 3100
-Wire Wire Line
-	4850 2950 4850 3100
+	4950 3100 4850 3100
+Wire Wire Line
+	4850 3100 4850 2950
 Wire Wire Line
 	5450 2300 5450 2400
@@
 Connection ~ 7200 4800
 Wire Wire Line
-	7200 4700 7200 4800
-Wire Wire Line
-	7300 4700 7200 4700
+	7200 4800 7200 4700
+Wire Wire Line
+	7200 4700 7300 4700
 Connection ~ 6000 4500
 Wire Wire Line
-	6000 4400 6000 4500
-Wire Wire Line
-	5900 4400 6000 4400
-Wire Wire Line
-	7200 4400 7200 4500
-Wire Wire Line
-	7300 4400 7200 4400
+	6000 4500 6000 4400
+Wire Wire Line
+	6000 4400 5900 4400
+Wire Wire Line
+	7200 4500 7200 4400
+Wire Wire Line
+	7200 4400 7300 4400
 Wire Wire Line
 	5900 4200 7300 4200
@@
 	7300 4800 5900 4800
 Wire Wire Line
-	6000 4700 5900 4700
-Wire Wire Line
-	6000 4800 6000 4700
+	5900 4700 6000 4700
+Wire Wire Line
+	6000 4700 6000 4800
 Connection ~ 6000 4800
 Wire Wire Line

Commit message: Did some silk work
git-svn-id: file:///home/ff/projects/osaa/svn@231 a092026d-3e22-4cff-94a7-eaa6fdd35d37
Connections:
- net GND: now also CON7.22 (shield), CON8.22 (shield)
Changed lines of the file:
@@
-EESchema Schematic File Version 2  date 2010-12-23T21:46:15 CET
+EESchema Schematic File Version 2  date 2010-12-25T12:56:58 CET
 LIBS:enc28j60
 LIBS:power
@@
 Sheet 3 6
 Title ""
-Date "23 dec 2010"
+Date "25 dec 2010"
 Rev ""
 Comp ""
@@
 Comment4 ""
 $EndDescr
+Wire Wire Line
+	7200 4950 7200 4700
+Wire Wire Line
+	7200 4950 7300 4950
+Wire Wire Line
+	3950 3600 3950 3700
+Wire Wire Line
+	3600 2750 4950 2750
+Wire Wire Line
+	4450 4150 4450 4000
+Wire Wire Line
+	4700 3600 4700 3700
+Connection ~ 4700 2600
+Wire Wire Line
+	4700 3100 4700 2600
+Wire Wire Line
+	4200 3700 4200 3600
+Connection ~ 4200 2950
+Wire Wire Line
+	4200 2950 4200 3100
+Connection ~ 6150 2700
+Wire Wire Line
+	5950 2700 6300 2700
+Wire Wire Line
+	7050 3000 6900 3000
+Wire Wire Line
+	7550 2700 7650 2700
+Wire Wire Line
+	7650 2700 7650 3250
+Connection ~ 6150 4500
+Wire Wire Line
+	6150 4450 6150 4500
+Wire Wire Line
+	4950 3100 4850 3100
+Wire Wire Line
+	4850 3100 4850 2950
+Wire Wire Line
+	5450 2300 5450 2400
+Connection ~ 6050 4100
+Wire Wire Line
+	6050 3000 6050 4100
+Wire Wire Line
+	5900 4600 7300 4600
+Connection ~ 7200 4800
+Wire Wire Line
+	7200 4700 7300 4700
+Connection ~ 6000 4500
+Wire Wire Line
+	6000 4500 6000 4400
+Wire Wire Line
+	6000 4400 5900 4400
+Wire Wire Line
+	7200 4500 7200 4400
+Wire Wire Line
+	7200 4400 7300 4400
+Wire Wire Line
+	5900 4200 7300 4200
+Wire Wire Line
+	7300 4100 5900 4100
+Wire Wire Line
+	5900 4300 7300 4300
+Wire Wire Line
+	7300 4500 5900 4500
+Connection ~ 7200 4500
+Wire Wire Line
+	7300 4800 5900 4800
+Wire Wire Line
+	5900 4700 6000 4700
+Connection ~ 6000 4800
+Wire Wire Line
+	6150 4200 6150 2700
+Connection ~ 6150 4200
+Wire Wire Line
+	5450 3400 5450 3300
+Connection ~ 4850 2950
+Wire Wire Line
+	4950 2600 3600 2600
+Wire Wire Line
+	6150 4800 6150 4900
+Connection ~ 6150 4800
+Wire Wire Line
+	7550 3000 7650 3000
+Connection ~ 7650 3000
+Wire Wire Line
+	7050 2700 6900 2700
+Wire Wire Line
+	5950 3000 6300 3000
+Connection ~ 6050 3000
+Wire Wire Line
+	4200 4000 4200 4150
+Wire Wire Line
+	4450 2750 4450 3100
+Connection ~ 4450 2750
+Wire Wire Line
+	4450 3600 4450 3700
+Wire Wire Line
+	4700 4000 4700 4150
+Wire Wire Line
+	3600 2950 4950 2950
+Wire Wire Line
+	3600 3100 3950 3100
+Wire Wire Line
+	3950 4000 3950 4150
+Wire Wire Line
+	5900 4950 6000 4950
+Wire Wire Line
+	6000 4950 6000 4700
 $Comp
 L +5V #PWR037
@@
 Text Notes 5150 1600 0    60   ~ 0
 RS-485
-Wire Wire Line
-	3950 3600 3950 3700
-Wire Wire Line
-	3600 2750 4950 2750
-Wire Wire Line
-	4450 4150 4450 4000
-Wire Wire Line
-	4700 3600 4700 3700
-Connection ~ 4700 2600
-Wire Wire Line
-	4700 3100 4700 2600
-Wire Wire Line
-	4200 3700 4200 3600
-Connection ~ 4200 2950
-Wire Wire Line
-	4200 2950 4200 3100
-Connection ~ 6150 2700
-Wire Wire Line
-	5950 2700 6300 2700
-Wire Wire Line
-	7050 3000 6900 3000
-Wire Wire Line
-	7550 2700 7650 2700
-Wire Wire Line
-	7650 2700 7650 3250
-Connection ~ 6150 4500
-Wire Wire Line
-	6150 4450 6150 4500
-Wire Wire Line
-	4950 3100 4850 3100
-Wire Wire Line
-	4850 3100 4850 2950
-Wire Wire Line
-	5450 2300 5450 2400
-Connection ~ 6050 4100
-Wire Wire Line
-	6050 3000 6050 4100
-Wire Wire Line
-	5900 4600 7300 4600
-Connection ~ 7200 4800
-Wire Wire Line
-	7200 4800 7200 4700
-Wire Wire Line
-	7200 4700 7300 4700
-Connection ~ 6000 4500
-Wire Wire Line
-	6000 4500 6000 4400
-Wire Wire Line
-	6000 4400 5900 4400
-Wire Wire Line
-	7200 4500 7200 4400
-Wire Wire Line
-	7200 4400 7300 4400
-Wire Wire Line
-	5900 4200 7300 4200
-Wire Wire Line
-	7300 4100 5900 4100
-Wire Wire Line
-	5900 4300 7300 4300
-Wire Wire Line
-	7300 4500 5900 4500
-Connection ~ 7200 4500
-Wire Wire Line
-	7300 4800 5900 4800
-Wire Wire Line
-	5900 4700 6000 4700
-Wire Wire Line
-	6000 4700 6000 4800
-Connection ~ 6000 4800
-Wire Wire Line
-	6150 4200 6150 2700
-Connection ~ 6150 4200
-Wire Wire Line
-	5450 3400 5450 3300
-Connection ~ 4850 2950
-Wire Wire Line
-	4950 2600 3600 2600
-Wire Wire Line
-	6150 4800 6150 4900
-Connection ~ 6150 4800
-Wire Wire Line
-	7550 3000 7650 3000
-Connection ~ 7650 3000
-Wire Wire Line
-	7050 2700 6900 2700
-Wire Wire Line
-	5950 3000 6300 3000
-Connection ~ 6050 3000
-Wire Wire Line
-	4200 4000 4200 4150
-Wire Wire Line
-	4450 2750 4450 3100
-Connection ~ 4450 2750
-Wire Wire Line
-	4450 3600 4450 3700
-Wire Wire Line
-	4700 4000 4700 4150
-Wire Wire Line
-	3600 2950 4950 2950
-Wire Wire Line
-	3600 3100 3950 3100
-Wire Wire Line
-	3950 4000 3950 4150
 $EndSCHEMATC
