File: cerberus/hardware-4.0/doorctrl-rs485.sch (KiCad schematic (older format))
At the start: 11 parts, among them CON7 RJHSE-5085, CON8 RJHSE-5085, U7 sp485

Commit message: Various fixes
git-svn-id: file:///home/ff/projects/osaa/svn@236 a092026d-3e22-4cff-94a7-eaa6fdd35d37
Connections:
- net +5V: now also CON8.10 (A), CON8.12 (A)
- net GND: no longer CON8.11 (C), CON8.9 (C)
- net at R60.2: now also CON8.11 (C); no longer CON8.12 (A)
- net at R59.2: now also CON8.9 (C); no longer CON8.10 (A)
Other:
- moved on the sheet: CON8B, CON8C
Changed lines of the file:
@@
-EESchema Schematic File Version 2  date 2010-12-28T16:33:17 CET
+EESchema Schematic File Version 2  date 2011-01-01T13:33:03 CET
 LIBS:enc28j60
 LIBS:power
@@
 Sheet 3 6
 Title ""
-Date "28 dec 2010"
+Date "1 jan 2011"
 Rev ""
 Comp ""
@@
 Comment4 ""
 $EndDescr
+$Comp
+L +5V #PWR038
+U 1 1 4D1C8A60
+P 4700 4150
+F 0 "#PWR038" H 4700 4240 20  0001 C CNN
+F 1 "+5V" H 4700 4240 30  0000 C CNN
+	1    4700 4150
+	-1   0    0    1
+$EndComp
+$Comp
+L +5V #PWR039
+U 1 1 4D1C8A58
+P 4450 4150
+F 0 "#PWR039" H 4450 4240 20  0001 C CNN
+F 1 "+5V" H 4450 4240 30  0000 C CNN
+	1    4450 4150
+	-1   0    0    1
+$EndComp
+$Comp
+L RJHSE-5085 CON?
+U 3 1 4D0BB203
+P 4700 3900
+AR Path="/4CFD2FB8/4D0A7710" Ref="CON?"  Part="3"
+AR Path="/4D0BB1C7/4D0BB203" Ref="CON8"  Part="3"
+F 0 "CON8" V 4700 4450 60  0000 C CNN
+F 1 "RJHSE-5085" H 4800 4300 60  0001 C CNN
+	3    4700 3900
+	-1   0    0    1
+$EndComp
+Wire Wire Line
+	3600 2750 4950 2750
 Wire Wire Line
 	7200 4950 7200 4700
@@
 Wire Wire Line
 	3950 3600 3950 3700
-Wire Wire Line
-	3600 2750 4950 2750
 Wire Wire Line
 	4450 4150 4450 4000
@@
 	6000 4950 6000 4700
 $Comp
-L +5V #PWR038
+L +5V #PWR040
 U 1 1 4D0BB20A
 P 5450 2300
-F 0 "#PWR038" H 5450 2390 20  0001 C CNN
+F 0 "#PWR040" H 5450 2390 20  0001 C CNN
 F 1 "+5V" H 5450 2390 30  0000 C CNN
 	1    5450 2300
@@
 L RJHSE-5085 CON?
 U 2 1 4D0BB204
-P 4450 3800
+P 4450 3900
 AR Path="/4CFD2FB8/4D0A770C" Ref="CON?"  Part="2"
 AR Path="/4D0BB1C7/4D0BB204" Ref="CON8"  Part="2"
-F 0 "CON8" V 4450 3150 60  0000 C CNN
-F 1 "RJHSE-5085" H 4550 4200 60  0001 C CNN
-	2    4450 3800
-	1    0    0    -1
-$EndComp
-$Comp
-L RJHSE-5085 CON?
-U 3 1 4D0BB203
-P 4700 3800
-AR Path="/4CFD2FB8/4D0A7710" Ref="CON?"  Part="3"
-AR Path="/4D0BB1C7/4D0BB203" Ref="CON8"  Part="3"
-F 0 "CON8" V 4700 3150 60  0000 C CNN
-F 1 "RJHSE-5085" H 4800 4200 60  0001 C CNN
-	3    4700 3800
-	1    0    0    -1
-$EndComp
-$Comp
-L GND #PWR039
+F 0 "CON8" V 4450 4450 60  0000 C CNN
+F 1 "RJHSE-5085" H 4550 4300 60  0001 C CNN
+	2    4450 3900
+	-1   0    0    1
+$EndComp
+$Comp
+L GND #PWR041
 U 1 1 4D0BB201
 P 5450 3400
-F 0 "#PWR039" H 5450 3400 30  0001 C CNN
+F 0 "#PWR041" H 5450 3400 30  0001 C CNN
 F 1 "GND" H 5450 3330 30  0001 C CNN
 	1    5450 3400
@@
 TXENABLE
 $Comp
-L +24V #PWR040
+L +24V #PWR042
 U 1 1 4D0BB200
 P 6150 4450
-F 0 "#PWR040" H 6150 4400 20  0001 C CNN
+F 0 "#PWR042" H 6150 4400 20  0001 C CNN
 F 1 "+24V" H 6150 4550 30  0000 C CNN
 	1    6150 4450
@@
 $EndComp
 $Comp
-L GND #PWR041
+L GND #PWR043
 U 1 1 4D0BB1FF
 P 6150 4900
-F 0 "#PWR041" H 6150 4900 30  0001 C CNN
+F 0 "#PWR043" H 6150 4900 30  0001 C CNN
 F 1 "GND" H 6150 4830 30  0001 C CNN
 	1    6150 4900
@@
 $EndComp
 $Comp
-L GND #PWR042
+L GND #PWR044
 U 1 1 4D0BB1FA
 P 7650 3250
-F 0 "#PWR042" H 7650 3250 30  0001 C CNN
+F 0 "#PWR044" H 7650 3250 30  0001 C CNN
 F 1 "GND" H 7650 3180 30  0001 C CNN
 	1    7650 3250
@@
 Termination jumpers
 $Comp
-L GND #PWR043
+L GND #PWR045
 U 1 1 4D0BB1F9
 P 4200 4150
-F 0 "#PWR043" H 4200 4150 30  0001 C CNN
+F 0 "#PWR045" H 4200 4150 30  0001 C CNN
 F 1 "GND" H 4200 4080 30  0001 C CNN
 	1    4200 4150
@@
 	1    0    0    -1
 $EndComp
-$Comp
-L GND #PWR044
-U 1 1 4D0BB1F7
-P 4450 4150
-F 0 "#PWR044" H 4450 4150 30  0001 C CNN
-F 1 "GND" H 4450 4080 30  0001 C CNN
-	1    4450 4150
-	1    0    0    -1
-$EndComp
-$Comp
-L GND #PWR045
-U 1 1 4D0BB1F6
-P 4700 4150
-F 0 "#PWR045" H 4700 4150 30  0001 C CNN
-F 1 "GND" H 4700 4080 30  0001 C CNN
-	1    4700 4150
-	1    0    0    -1
-$EndComp
