File: cerberus/hardware-4.0/doorctrl-v4-net.sch (KiCad schematic (older format))
At the start: 37 parts, among them CON6 RJHSE-5085, U4 ENC28J60, U5 MC34063, X2 25MHz

Commit message: Added torroid coil and proper diode packages
git-svn-id: file:///home/ff/projects/osaa/svn@222 a092026d-3e22-4cff-94a7-eaa6fdd35d37
Parts:
- removed C38: 100uF, symbol CAPAPOL
- C44: value 100uF -> 100nF
Other:
- moved on the sheet: C39
Changed lines of the file:
@@
-EESchema Schematic File Version 2  date 2010-12-18T14:49:05 CET
+EESchema Schematic File Version 2  date 2010-12-19T21:45:09 CET
 LIBS:enc28j60
 LIBS:power
@@
 Sheet 2 6
 Title ""
-Date "18 dec 2010"
+Date "19 dec 2010"
 Rev ""
 Comp ""
@@
 Connection ~ 8050 6650
 Connection ~ 7550 6650
-Connection ~ 6850 6650
 Connection ~ 7350 5950
 Connection ~ 6550 6250
@@
 	5600 6400 5600 5950
 Connection ~ 6850 6250
-Connection ~ 7150 6250
 Connection ~ 6550 6650
-Connection ~ 7150 6650
+Connection ~ 6850 6650
 Connection ~ 7800 6650
 Connection ~ 7800 6250
@@
 Connection ~ 4750 1650
 Wire Wire Line
-	4750 1650 4750 1750
+	4750 1750 4750 1650
 Wire Wire Line
 	4650 1750 4650 1600
@@
 P 8550 6450
 F 0 "C44" H 8600 6550 50  0000 L CNN
-F 1 "100uF" H 8600 6350 50  0000 L CNN
+F 1 "100nF" H 8600 6350 50  0000 L CNN
 	1    8550 6450
 	1    0    0    -1
@@
 Distributed decoupling capacitors
 $Comp
-L GND #PWR32
+L GND #PWR016
 U 1 1 4D0BB162
 P 7350 6800
-F 0 "#PWR32" H 7350 6800 30  0001 C CNN
+F 0 "#PWR016" H 7350 6800 30  0001 C CNN
 F 1 "GND" H 7350 6730 30  0001 C CNN
 	1    7350 6800
@@
 L C C39
 U 1 1 4D0BB15D
-P 7150 6450
-F 0 "C39" H 7200 6550 50  0000 L CNN
-F 1 "10uF" H 7200 6350 50  0000 L CNN
-	1    7150 6450
-	1    0    0    -1
-$EndComp
-$Comp
-L +3.3V #PWR31
+P 6850 6450
+F 0 "C39" H 6900 6550 50  0000 L CNN
+F 1 "10uF" H 6900 6350 50  0000 L CNN
+	1    6850 6450
+	1    0    0    -1
+$EndComp
+$Comp
+L +3.3V #PWR017
 U 1 1 4D0BB15C
 P 7350 5850
-F 0 "#PWR31" H 7350 5810 30  0001 C CNN
+F 0 "#PWR017" H 7350 5810 30  0001 C CNN
 F 1 "+3.3V" H 7350 5960 30  0000 C CNN
 	1    7350 5850
-	1    0    0    -1
-$EndComp
-$Comp
-L CAPAPOL C38
-U 1 1 4D0BB15B
-P 6850 6450
-F 0 "C38" H 6900 6550 50  0000 L CNN
-F 1 "100uF" H 6900 6350 50  0000 L CNN
-	1    6850 6450
 	1    0    0    -1
 $EndComp
@@
 $EndComp
 $Comp
-L GND #PWR17
+L GND #PWR018
 U 1 1 4D0BB156
 P 3700 7100
-F 0 "#PWR17" H 3700 7100 30  0001 C CNN
+F 0 "#PWR018" H 3700 7100 30  0001 C CNN
 F 1 "GND" H 3700 7030 30  0001 C CNN
 	1    3700 7100
@@
 $EndComp
 $Comp
-L GND #PWR25
+L GND #PWR019
 U 1 1 4D0BB155
 P 5400 7100
-F 0 "#PWR25" H 5400 7100 30  0001 C CNN
+F 0 "#PWR019" H 5400 7100 30  0001 C CNN
 F 1 "GND" H 5400 7030 30  0001 C CNN
 	1    5400 7100
@@
 $EndComp
 $Comp
-L GND #PWR21
+L GND #PWR020
 U 1 1 4D0BB154
 P 4550 6800
-F 0 "#PWR21" H 4550 6800 30  0001 C CNN
+F 0 "#PWR020" H 4550 6800 30  0001 C CNN
 F 1 "GND" H 4550 6730 30  0001 C CNN
 	1    4550 6800
@@
 $EndComp
 $Comp
-L +24V #PWR20
+L +24V #PWR021
 U 1 1 4D0BB150
 P 4550 5600
-F 0 "#PWR20" H 4550 5550 20  0001 C CNN
+F 0 "#PWR021" H 4550 5550 20  0001 C CNN
 F 1 "+24V" H 4550 5700 30  0000 C CNN
 	1    4550 5600
@@
 $EndComp
 $Comp
-L +24V #PWR34
+L +24V #PWR022
 U 1 1 4D09235E
 P 7925 3525
-F 0 "#PWR34" H 7925 3475 20  0001 C CNN
+F 0 "#PWR022" H 7925 3475 20  0001 C CNN
 F 1 "+24V" H 7925 3625 30  0000 C CNN
 	1    7925 3525
@@
 $EndComp
 $Comp
-L GND #PWR35
+L GND #PWR023
 U 1 1 4D092355
 P 8050 3950
-F 0 "#PWR35" H 8050 3950 30  0001 C CNN
+F 0 "#PWR023" H 8050 3950 30  0001 C CNN
 F 1 "GND" H 8050 3880 30  0001 C CNN
 	1    8050 3950
@@
 $EndComp
 $Comp
-L GND #PWR33
+L GND #PWR024
 U 1 1 4D09232A
 P 7725 4950
-F 0 "#PWR33" H 7725 4950 30  0001 C CNN
+F 0 "#PWR024" H 7725 4950 30  0001 C CNN
 F 1 "GND" H 7725 4880 30  0001 C CNN
 	1    7725 4950
@@
 $EndComp
 $Comp
-L GND #PWR27
+L GND #PWR025
 U 1 1 4D09222A
 P 5600 3350
-F 0 "#PWR27" H 5600 3350 30  0001 C CNN
+F 0 "#PWR025" H 5600 3350 30  0001 C CNN
 F 1 "GND" H 5600 3280 30  0001 C CNN
 	1    5600 3350
@@
 $EndComp
 $Comp
-L +3.3V #PWR29
+L +3.3V #PWR026
 U 1 1 4D092180
 P 6150 1450
-F 0 "#PWR29" H 6150 1410 30  0001 C CNN
+F 0 "#PWR026" H 6150 1410 30  0001 C CNN
 F 1 "+3.3V" H 6150 1560 30  0000 C CNN
 	1    6150 1450
@@
 $EndComp
 $Comp
-L GND #PWR26
+L GND #PWR027
 U 1 1 4D0920F3
 P 5600 2550
-F 0 "#PWR26" H 5600 2550 30  0001 C CNN
+F 0 "#PWR027" H 5600 2550 30  0001 C CNN
 F 1 "GND" H 5600 2480 30  0001 C CNN
 	1    5600 2550
@@
 $EndComp
 $Comp
-L +3.3V #PWR19
+L +3.3V #PWR028
 U 1 1 4D091E1A
 P 4050 1600
-F 0 "#PWR19" H 4050 1560 30  0001 C CNN
+F 0 "#PWR028" H 4050 1560 30  0001 C CNN
 F 1 "+3.3V" H 4050 1710 30  0000 C CNN
 	1    4050 1600
@@
 $EndComp
 $Comp
-L GND #PWR30
+L GND #PWR029
 U 1 1 4D091D90
 P 6500 4700
-F 0 "#PWR30" H 6500 4700 30  0001 C CNN
+F 0 "#PWR029" H 6500 4700 30  0001 C CNN
 F 1 "GND" H 6500 4630 30  0001 C CNN
 	1    6500 4700
@@
 $EndComp
 $Comp
-L GND #PWR28
+L GND #PWR030
 U 1 1 4D091D8C
 P 5600 4700
-F 0 "#PWR28" H 5600 4700 30  0001 C CNN
+F 0 "#PWR030" H 5600 4700 30  0001 C CNN
 F 1 "GND" H 5600 4630 30  0001 C CNN
 	1    5600 4700
@@
 $EndComp
 $Comp
-L GND #PWR18
+L GND #PWR031
 U 1 1 4D091D21
 P 4000 4300
-F 0 "#PWR18" H 4000 4300 30  0001 C CNN
+F 0 "#PWR031" H 4000 4300 30  0001 C CNN
 F 1 "GND" H 4000 4230 30  0001 C CNN
 	1    4000 4300
@@
 $EndComp
 $Comp
-L GND #PWR16
+L GND #PWR032
 U 1 1 4D091D1E
 P 3700 4300
-F 0 "#PWR16" H 3700 4300 30  0001 C CNN
+F 0 "#PWR032" H 3700 4300 30  0001 C CNN
 F 1 "GND" H 3700 4230 30  0001 C CNN
 	1    3700 4300
@@
 $EndComp
 $Comp
-L GND #PWR15
+L GND #PWR033
 U 1 1 4D091D1B
 P 3500 4300
-F 0 "#PWR15" H 3500 4300 30  0001 C CNN
+F 0 "#PWR033" H 3500 4300 30  0001 C CNN
 F 1 "GND" H 3500 4230 30  0001 C CNN
 	1    3500 4300
@@
 Clock out
 $Comp
-L GND #PWR24
+L GND #PWR034
 U 1 1 4D091ABE
 P 5250 1050
-F 0 "#PWR24" H 5250 1050 30  0001 C CNN
+F 0 "#PWR034" H 5250 1050 30  0001 C CNN
 F 1 "GND" H 5250 980 30  0001 C CNN
 	1    5250 1050
@@
 $EndComp
 $Comp
-L GND #PWR23
+L GND #PWR035
 U 1 1 4D0919DD
 P 4650 4450
-F 0 "#PWR23" H 4650 4450 30  0001 C CNN
+F 0 "#PWR035" H 4650 4450 30  0001 C CNN
 F 1 "GND" H 4650 4380 30  0001 C CNN
 	1    4650 4450
@@
 $EndComp
 $Comp
-L +3.3V #PWR22
+L +3.3V #PWR036
 U 1 1 4D0919D8
 P 4650 1600
-F 0 "#PWR22" H 4650 1560 30  0001 C CNN
+F 0 "#PWR036" H 4650 1560 30  0001 C CNN
 F 1 "+3.3V" H 4650 1710 30  0000 C CNN
 	1    4650 1600

Commit message: Started laying out the PCB for real
git-svn-id: file:///home/ff/projects/osaa/svn@223 a092026d-3e22-4cff-94a7-eaa6fdd35d37
Parts:
- U4: footprint SSOP28 -> (none)
Connections:
- net rd+: now reaches R48.2, TX1.16 (RD+), U4.12 (TPIN-)
- net rd-: now reaches R47.2, TX1.15 (RD-), U4.13 (TPIN+)
- net td+: now reaches R46.2, TX1.1 (TD+), U4.16 (TPOUT-)
- net td-: now reaches R45.2, TX1.2 (TD-), U4.17 (TPOUT+)
- net tx-: now reaches CON6.1, TX1.7 (TX-)
- net tx+: now reaches CON6.2, TX1.8 (TX+)
- net rx-: now reaches CON6.3, TX1.10 (RX-)
- net rx+: now reaches CON6.6, TX1.9 (RX+)
- net rxct: now reaches R49.1, TX1.11 (RXCT)
- net tct: now reaches C32.1, L3.2, R45.1, R46.1, TX1.3 (TCT)
- net txct: now reaches R50.1, TX1.6 (TXCT)
Changed lines of the file:
@@
-EESchema Schematic File Version 2  date 2010-12-19T21:45:09 CET
+EESchema Schematic File Version 2  date 2010-12-20T22:26:04 CET
 LIBS:enc28j60
 LIBS:power
@@
 LIBS:linear
 LIBS:atmel
+LIBS:diode
 LIBS:doorctrl-v4-cache
 EELAYER 24  0
@@
 Sheet 2 6
 Title ""
-Date "19 dec 2010"
+Date "20 dec 2010"
 Rev ""
 Comp ""
@@
 Comment4 ""
 $EndDescr
+Text Label 6350 3650 0    60   ~ 0
+rd+
+Text Label 6350 3050 0    60   ~ 0
+rd-
+Text Label 6350 2850 0    60   ~ 0
+td+
+Text Label 6350 2550 0    60   ~ 0
+tct
+Text Label 6350 2250 0    60   ~ 0
+td-
+Text Label 7650 3650 0    60   ~ 0
+rx+
+Text Label 7600 3350 0    60   ~ 0
+rxct
+Text Label 7650 3050 0    60   ~ 0
+rx-
+Text Label 7650 2850 0    60   ~ 0
+tx+
+Text Label 7650 2550 0    60   ~ 0
+txct
+Text Label 7650 2250 0    60   ~ 0
+tx-
 Text Notes 750  7600 0    60   ~ 0
 All these parts are optional and only needed if Ethernet is wanted
@@
 F 0 "U4" H 4765 2350 50  0000 L BNN
 F 1 "ENC28J60" H 4750 3350 50  0000 L BNN
-F 2 "SSOP28" H 4850 3100 50  0001 C CNN
 	1    4850 2950
 	1    0    0    -1

Commit message: Converted to 2010-12-18
git-svn-id: file:///home/ff/projects/osaa/svn@225 a092026d-3e22-4cff-94a7-eaa6fdd35d37
Connections:
- net Clock out renamed Clock-out
Changed lines of the file:
@@
-EESchema Schematic File Version 2  date 2010-12-20T22:26:04 CET
+EESchema Schematic File Version 2  date 2010-12-21T17:47:20 CET
 LIBS:enc28j60
 LIBS:power
@@
 Sheet 2 6
 Title ""
-Date "20 dec 2010"
+Date "21 dec 2010"
 Rev ""
 Comp ""
@@
 ~CS
 Text HLabel 4000 2550 0    60   Output ~ 0
-Clock out
+Clock-out
 $Comp
 L GND #PWR034

Commit message: Finished the copper layers
git-svn-id: file:///home/ff/projects/osaa/svn@229 a092026d-3e22-4cff-94a7-eaa6fdd35d37
Connections:
- net vcap: now reaches C30.1, U4.1 (VCAP)
- net ~enc-reset: now reaches R42.2, U4.10 (!RESET)
- net rbias: now reaches R40.1, R41.1, U4.14 (RBIAS)
- net osc1: now reaches C34.1, U4.23 (OSC1), X2.2
- net osc2: now reaches C31.1, U4.24 (OSC2), X2.1
- net Clock-out: no longer names the net of U4.3 (CLKOUT)
Changed lines of the file:
@@
-EESchema Schematic File Version 2  date 2010-12-21T17:47:20 CET
+EESchema Schematic File Version 2  date 2010-12-23T21:46:15 CET
 LIBS:enc28j60
 LIBS:power
@@
 LIBS:diode
 LIBS:doorctrl-v4-cache
-EELAYER 24  0
+EELAYER 25  0
 EELAYER END
 $Descr A4 11700 8267
 Sheet 2 6
 Title ""
-Date "21 dec 2010"
+Date "23 dec 2010"
 Rev ""
 Comp ""
@@
 Comment4 ""
 $EndDescr
+Text Label 4050 2450 2    60   ~ 0
+~enc-reset
+Text Label 5500 4050 0    60   ~ 0
+osc2
+Text Label 5500 3850 0    60   ~ 0
+osc1
+Text Label 3700 3550 0    60   ~ 0
+rbias
+Text Label 4000 3650 0    60   ~ 0
+vcap
 Text Label 6350 3650 0    60   ~ 0
 rd+
@@
 Connection ~ 4550 1650
 Wire Wire Line
-	4000 2550 4250 2550
-Wire Wire Line
 	4250 2950 4000 2950
 Wire Wire Line
@@
 Text HLabel 4000 2850 0    60   Input ~ 0
 ~CS
-Text HLabel 4000 2550 0    60   Output ~ 0
-Clock-out
 $Comp
 L GND #PWR034

Commit message: Did some silk work
git-svn-id: file:///home/ff/projects/osaa/svn@231 a092026d-3e22-4cff-94a7-eaa6fdd35d37
Connections:
- net GND: now also CON6.22 (shield)

Commit message: Various tweakage
git-svn-id: file:///home/ff/projects/osaa/svn@233 a092026d-3e22-4cff-94a7-eaa6fdd35d37
Connections:
- no-connect marks 0 -> 4
Changed lines of the file:
@@
-EESchema Schematic File Version 2  date 2010-12-25T12:56:58 CET
+EESchema Schematic File Version 2  date 2010-12-27T14:47:10 CET
 LIBS:enc28j60
 LIBS:power
@@
 Sheet 2 6
 Title ""
-Date "25 dec 2010"
+Date "27 dec 2010"
 Rev ""
 Comp ""
@@
 Comment4 ""
 $EndDescr
+NoConn ~ 4250 3350
+NoConn ~ 4250 2650
+NoConn ~ 4250 2550
+NoConn ~ 6600 3350
 Connection ~ 8050 4000
 Wire Wire Line
