File: cerberus/hardware-4/doorctrl-rs485.sch (KiCad schematic (older format))
At the start: 11 parts, among them CON7 RJHSE-5085, CON8 RJHSE-5085, U7 sp485

Commit message: Various cleanups
git-svn-id: file:///home/ff/projects/osaa/svn@255 a092026d-3e22-4cff-94a7-eaa6fdd35d37
Parts:
- U7: value sp485 -> DS75176BM
Changed lines of the file:
@@
-EESchema Schematic File Version 2  date 2011-01-03T16:40:54 CET
+EESchema Schematic File Version 2  date 2011-01-17T19:42:11 CET
 LIBS:enc28j60
 LIBS:power
@@
 Sheet 3 6
 Title ""
-Date "3 jan 2011"
+Date "17 jan 2011"
 Rev ""
 Comp ""
@@
 P 5450 2850
 F 0 "U7" H 5450 2950 60  0000 C CNN
-F 1 "sp485" H 5450 2850 60  0000 C CNN
+F 1 "DS75176BM" H 5450 2850 60  0000 C CNN
 F 2 "so8" H 5650 2600 60  0001 C CNN
 	1    5450 2850
