File: cerberus/hardware-4/doorctrl-v4-rfid.sch (KiCad schematic (older format))
At the start: 19 parts, among them Q1 BC817, Q2 BC807, U1 LM358

Commit message: Various fiddeling
git-svn-id: file:///home/ff/projects/osaa/svn@243 a092026d-3e22-4cff-94a7-eaa6fdd35d37
Other:
- note added: "Notice: If the RFID option is mounted on the board, then R22 and R23 must not be mounted."
Changed lines of the file:
@@
-EESchema Schematic File Version 2  date 2011-01-03T13:24:02 CET
+EESchema Schematic File Version 2  date 2011-01-03T16:40:54 CET
 LIBS:enc28j60
 LIBS:power
@@
 Comment4 ""
 $EndDescr
+Text Notes 750  7550 0    60   ~ 0
+Notice: If the RFID option is mounted on the board, then R22 and R23 must not be mounted.
 Wire Wire Line
 	4050 2900 5000 2900
