File: cerberus/hardware-4/doorctrl-v4.sch (KiCad schematic (older format))
At the start: 11 parts, among them CON1 ISP, CON10 5x2 header, CON2 JTAG, CON9 FTDI-serial, IC1 ATMEGA324P-A, U8 24LC64, X1 20MHz

Commit message: Various cleanups
git-svn-id: file:///home/ff/projects/osaa/svn@255 a092026d-3e22-4cff-94a7-eaa6fdd35d37
Parts:
- C1, C2: value 16pF -> 15pF
Other:
- note added: "Ethernet ~CS"
- note added: "SCL"
- note added: "SDA"
- moved on the sheet: CON1, CON2

Commit message: Fixed a couple of bugs: No more level shifter and rfid carrier wave output is connected correctly
git-svn-id: file:///home/ff/projects/osaa/svn@258 a092026d-3e22-4cff-94a7-eaa6fdd35d37
Connections:
- net PB1: now also CON10.9
- net PB3: no longer CON10.9
Changed lines of the file:
@@
-EESchema Schematic File Version 2  date 2011-01-17T20:19:18 CET
+EESchema Schematic File Version 2  date 2011-01-23T22:09:23 CET
 LIBS:enc28j60
 LIBS:power
@@
 Sheet 1 6
 Title ""
-Date "17 jan 2011"
+Date "23 jan 2011"
 Rev ""
 Comp ""
@@
 +3.3V
 Text GLabel 1200 6425 0    60   Input ~ 0
-PB3
+PB1
 Text GLabel 2100 6325 2    60   Input ~ 0
 PB2
@@
 Text Notes 4475 4500 0    60   ~ 0
 RFID - demodulated
-Text Notes 4475 2200 0    60   ~ 0
+Text Notes 4475 2400 0    60   ~ 0
 RFID carrier (125 kHz)
 Text Notes 4475 3500 0    60   ~ 0
@@
 PD6
 Text GLabel 9100 3875 0    60   Input ~ 0
-PB1
+PB3
 Text GLabel 9100 2700 0    60   Input ~ 0
 PB4
